Commit message: update urdf

File: pan_tilt_description/urdf/pan_tilt.urdf.xacro (robot description, xacro)
@@ -32,5 +32,5 @@
     </link>
     <joint name="${prefix}_yaw_joint" type="continuous">
-      <origin xyz="0.0 0.0 0.083" rpy="0.0 0.0 0.0"/>
+      <origin xyz="0.0 0.0 0.05455" rpy="0.0 0.0 0.0"/>
       <parent link="${prefix}_base_link"/>
       <child link="${prefix}_yaw_link"/>
@@ -50,5 +50,5 @@
     </link>
     <joint name="${prefix}_pitch_joint" type="continuous">
-      <origin xyz="0.0 0.0 0.060" rpy="0.0 0.0 0.0"/>
+      <origin xyz="0.0 0.0 0.057" rpy="0.0 0.0 0.0"/>
       <parent link="${prefix}_yaw_link"/>
       <child link="${prefix}_pitch_link"/>
@@ -58,5 +58,5 @@
     <link name="${prefix}_kinect_surface"/>
     <joint name="${prefix}_kinect_surface_joint" type="fixed">
-      <origin xyz="-0.0063 -0.010 -0.025" rpy="0 0 0" />
+      <origin xyz="0.0010 0.0077 -0.022" rpy="0 0 0" />
       <parent link="${prefix}_pitch_link"/>
       <child link="${prefix}_kinect_surface"/>

Commit message: fix file name, add kinect urdf

File: pan_tilt_description/urdf/pan_tilt.urdf.xacro (robot description, xacro)
@@ -13,5 +13,5 @@
         <origin xyz="0 0 0" rpy="0 0 0" />
         <geometry>
-          <mesh filename="package://pan_tilt_description/urdf/mesh/base.stl" />
+          <mesh filename="package://pan_tilt_description/mesh/base.stl" />
         </geometry>
         <material name="">
@@ -24,5 +24,5 @@
         <origin xyz="0 0 0" rpy="0 0 0" />
         <geometry>
-          <mesh filename="package://pan_tilt_description/urdf/mesh/pan.stl" />
+          <mesh filename="package://pan_tilt_description/mesh/pan.stl" />
         </geometry>
         <material name="">
@@ -31,5 +31,5 @@
       </visual>
     </link>
-    <joint name="${prefix}_yaw_joint" type="continuous">
+    <joint name="${prefix}_yaw_joint" type="revolute">
       <origin xyz="0.0 0.0 0.05455" rpy="0.0 0.0 0.0"/>
       <parent link="${prefix}_base_link"/>
@@ -42,5 +42,5 @@
         <origin xyz="0 0 0" rpy="0 0 0" />
         <geometry>
-          <mesh filename="package://pan_tilt_description/urdf/mesh/tilt.stl" />
+          <mesh filename="package://pan_tilt_description/mesh/tilt.stl" />
         </geometry>
         <material name="">
@@ -49,5 +49,5 @@
       </visual>
     </link>
-    <joint name="${prefix}_pitch_joint" type="continuous">
+    <joint name="${prefix}_pitch_joint" type="revolute">
       <origin xyz="0.0 0.0 0.057" rpy="0.0 0.0 0.0"/>
       <parent link="${prefix}_yaw_link"/>
