Commit message: fix kinect2_link pose

File: pan_tilt_description/urdf/kinect_v2.urdf.xacro (robot description, xacro)
@@ -21,5 +21,5 @@
     <link name="kinect2_link"/>
     <joint name="${prefix}_joint" type="fixed">
-      <origin xyz="0.01 -0.097 0.045" rpy="${-pi/2} 0 ${-pi/2}" />
+      <origin xyz="0.025 -0.05 0.049" rpy="${-pi/2} 0 ${-pi/2}" />
       <parent link="${prefix}_base"/>
       <child link="kinect2_link"/>
